Commit message: 로봇 기본 프레임 base_link -> base_footprint 변경

File: src/scout_description/urdf/scout_mini/scout_mini.xacro (robot description, xacro)
@@ -10,9 +10,9 @@
     <xacro:property name="track" value="0.49" />
     <xacro:property name="wheel_vertical_offset" value="-0.0905" />
-    <xacro:property name="wheel_length" value="0.8520e-01" />
-    <xacro:property name="wheel_radius" value="0.8750e-01" />
+    <xacro:property name="wheel_length" value="0.08520" />
+    <xacro:property name="wheel_radius" value="0.08750" />
     <link name="base_link">
         <visual>
-            <origin xyz="0 0 0" rpy="1.5707 0 1.5707" />
+            <origin xyz="0 0 0" rpy="0 0 0" />
             <geometry>
                 <mesh filename="package://scout_description/meshes/scout_mini/mini_base_link.dae" />
@@ -28,7 +28,7 @@
     <link name="base_footprint"/>
     <joint name="base_footprint_joint" type="fixed">
-        <origin xyz="0 0 ${wheel_vertical_offset - wheel_radius}" rpy="0 0 0" />
-        <parent link="base_link" />
-        <child link="base_footprint" />
+        <origin xyz="0 0 ${wheel_radius - wheel_vertical_offset}" rpy="0 0 0" />
+        <parent link="base_footprint" />
+        <child link="base_link" />
     </joint>
     <link name="inertial_link">
@@ -44,17 +44,4 @@
         <child link="inertial_link" />
     </joint>
-    <xacro:scout_mini_wheel wheel_prefix="front_right">
-        <origin xyz="${wheelbase/2} ${-track/2} ${wheel_vertical_offset}" rpy="0 0 -1.5707" />
-    </xacro:scout_mini_wheel>
-    <xacro:scout_mini_wheel wheel_prefix="front_left">
-        <origin xyz="${wheelbase/2} ${track/2} ${wheel_vertical_offset}" rpy="0 0 1.5707" />
-    </xacro:scout_mini_wheel>
-    <xacro:scout_mini_wheel wheel_prefix="rear_left">
-        <origin xyz="${-wheelbase/2} ${track/2} ${wheel_vertical_offset}" rpy="0 0 1.5707" />
-    </xacro:scout_mini_wheel>
-    <xacro:scout_mini_wheel wheel_prefix="rear_right">
-        <origin xyz="${-wheelbase/2} ${-track/2} ${wheel_vertical_offset}" rpy="0 0 -1.5707" />
-    </xacro:scout_mini_wheel>
-        <!-- Velodyne LiDAR -->
     <link name="velodyne_link">
         <visual>
@@ -63,30 +50,53 @@
                 <cylinder radius="0.05" length="0.08"/>
             </geometry>
-            <material name="black">
-                <color rgba="0.1 0.1 0.1 1.0"/>
+            <material name="velodyne_black">
+                <color rgba="0.02 0.02 0.02 1.0"/>
             </material>
         </visual>
+        <collision>
+            <origin xyz="0 0 0" rpy="0 0 0"/>
+            <geometry>
+                <cylinder radius="0.05" length="0.08"/>
+            </geometry>
+        </collision>
     </link>
     <joint name="velodyne_joint" type="fixed">
-        <origin xyz="0.0 0.0 0.5" rpy="0 0 0"/>
+        <origin xyz="0.0 0.0 0.45" rpy="0 0 0"/>
         <parent link="base_link"/>
         <child link="velodyne_link"/>
     </joint>
-    <!-- Intel RealSense Camera -->
     <link name="camera_link">
         <visual>
-            <origin xyz="0 0 0" rpy="0 0 0"/>
+            <origin xyz="0 0 0" rpy="0 0 1.5708"/>
             <geometry>
                 <box size="0.09 0.025 0.025"/>
             </geometry>
-            <material name="blue">
-                <color rgba="0.1 0.1 0.8 1.0"/>
+            <material name="camera_gray">
+                <color rgba="0.3 0.3 0.3 1.0"/>
             </material>
         </visual>
+        <collision>
+            <origin xyz="0 0 0" rpy="0 0 1.5708"/>
+            <geometry>
+                <box size="0.09 0.025 0.025"/>
+            </geometry>
+        </collision>
     </link>
     <joint name="camera_joint" type="fixed">
-        <origin xyz="0.20 0.0 0.24" rpy="0 0 0"/>
+        <origin xyz="0.24 0 0.04" rpy="0 0 0"/>
         <parent link="base_link"/>
         <child link="camera_link"/>
     </joint>
+    <xacro:scout_mini_wheel wheel_prefix="front_right">
+        <origin xyz="${wheelbase/2} ${-track/2} ${wheel_vertical_offset}" rpy="3.14 0 0" />
+    </xacro:scout_mini_wheel>
+    <xacro:scout_mini_wheel wheel_prefix="front_left">
+        <origin xyz="${wheelbase/2} ${track/2} ${wheel_vertical_offset}" rpy="0 0 0" />
+    </xacro:scout_mini_wheel>
+    <xacro:scout_mini_wheel wheel_prefix="rear_left">
+        <origin xyz="${-wheelbase/2} ${track/2} ${wheel_vertical_offset}" rpy="0 0 0" />
+    </xacro:scout_mini_wheel>
+    <xacro:scout_mini_wheel wheel_prefix="rear_right">
+        <origin xyz="${-wheelbase/2} ${-track/2} ${wheel_vertical_offset}" rpy="3.14 0 0" />
+    </xacro:scout_mini_wheel>
 </robot>

File: src/scout_description/urdf/scout_mini/scout_mini_wheel.xacro (robot description, xacro)
@@ -32,5 +32,5 @@
             </inertial>
             <visual>
-                <!-- <origin xyz="0 0 0" rpy="0 0 0" /> -->
+                <!--origin xyz="0 0 0" rpy="0 0 0" /-->
                 <origin xyz="${-0.452/2 + 0.005} ${-0.49/2 + 0.02} 0.0925" rpy="0 0 0" />
                 <geometry>
